File: Circuit/RotarySW.sch (KiCad schematic (older format))
At the start: 5 parts

Commit message: 部品の割り付け
Parts:
- gave numbers to parts that had none: 5
Changed lines of the file:
@@
 $Descr A4 11693 8268
 encoding utf-8
-Sheet 5 4
+Sheet 4 4
 Title ""
 Date ""
@@
 $EndDescr
 $Comp
-L SW_ROTARY SW?
+L SW_ROTARY SW1
 U 1 1 5936F68D
 P 6400 2950
-F 0 "SW?" H 6400 2950 60  0000 C CNN
+F 0 "SW1" H 6400 2950 60  0000 C CNN
 F 1 "SW_ROTARY" H 6400 2750 60  0000 C CNN
 F 2 "YASU:RotarySW" H 6400 2950 60  0001 C CNN
@@
 $EndComp
 $Comp
-L +3.3V #PWR018
+L +3.3V #PWR034
 U 1 1 5936F694
 P 5650 2250
-F 0 "#PWR018" H 5650 2100 50  0001 C CNN
+F 0 "#PWR034" H 5650 2100 50  0001 C CNN
 F 1 "+3.3V" H 5650 2390 50  0000 C CNN
 F 2 "" H 5650 2250 50  0000 C CNN
@@
 $EndComp
 $Comp
-L GND #PWR019
+L GND #PWR035
 U 1 1 5936F69A
 P 5650 3250
-F 0 "#PWR019" H 5650 3000 50  0001 C CNN
+F 0 "#PWR035" H 5650 3000 50  0001 C CNN
 F 1 "GND" H 5650 3100 50  0000 C CNN
 F 2 "" H 5650 3250 50  0000 C CNN
@@
 $EndComp
 $Comp
-L R R?
+L R R7
 U 1 1 5936F6A0
 P 5650 2550
-F 0 "R?" V 5730 2550 50  0000 C CNN
+F 0 "R7" V 5730 2550 50  0000 C CNN
 F 1 "10k" V 5650 2550 50  0000 C CNN
 F 2 "Resistors_SMD:R_0603_HandSoldering" V 5580 2550 50  0001 C CNN
@@
 $EndComp
 $Comp
-L R R?
+L R R6
 U 1 1 5936F6A7
 P 5500 2550
-F 0 "R?" V 5580 2550 50  0000 C CNN
+F 0 "R6" V 5580 2550 50  0000 C CNN
 F 1 "10k" V 5500 2550 50  0000 C CNN
 F 2 "Resistors_SMD:R_0603_HandSoldering" V 5430 2550 50  0001 C CNN
@@
 $EndComp
 $Comp
-L R R?
+L R R5
 U 1 1 5936F6AE
 P 5350 2550
-F 0 "R?" V 5430 2550 50  0000 C CNN
+F 0 "R5" V 5430 2550 50  0000 C CNN
 F 1 "10k" V 5350 2550 50  0000 C CNN
 F 2 "Resistors_SMD:R_0603_HandSoldering" V 5280 2550 50  0001 C CNN
@@
 $EndComp
 $Comp
-L R R?
+L R R4
 U 1 1 5936F6B5
 P 5200 2550
-F 0 "R?" V 5280 2550 50  0000 C CNN
+F 0 "R4" V 5280 2550 50  0000 C CNN
 F 1 "10k" V 5200 2550 50  0000 C CNN
 F 2 "Resistors_SMD:R_0603_HandSoldering" V 5130 2550 50  0001 C CNN
@@
 	5500 2700 5500 2950
 Wire Wire Line
-	5750 2950 5500 2950
-Wire Wire Line
-	5500 2950 4950 2950
+	4950 2950 5750 2950
 Wire Wire Line
 	5350 2700 5350 3050
 Wire Wire Line
-	5750 3050 5350 3050
-Wire Wire Line
-	5350 3050 4950 3050
+	4950 3050 5750 3050
 Wire Wire Line
 	5200 2700 5200 3150
 Wire Wire Line
-	5750 3150 5200 3150
-Wire Wire Line
-	5200 3150 4950 3150
+	4950 3150 5750 3150
 Connection ~ 5200 3150
 Connection ~ 5350 3050
@@
 Connection ~ 5650 2750
 Wire Wire Line
-	5650 2400 5650 2350
-Wire Wire Line
-	5650 2350 5650 2250
+	5650 2250 5650 2400
 Wire Wire Line
 	5200 2400 5200 2350
 Wire Wire Line
-	5200 2350 5350 2350
-Wire Wire Line
-	5350 2350 5500 2350
-Wire Wire Line
-	5500 2350 5650 2350
+	5200 2350 5650 2350
 Connection ~ 5650 2350
 Wire Wire Line
@@
 Connection ~ 5350 2350
 Wire Wire Line
-	5750 2750 5650 2750
-Wire Wire Line
-	5650 2750 4950 2750
+	4950 2750 5750 2750
 Text HLabel 4950 3150 0    60   Output ~ 0
 BIT0
