File: Circuit/Left_Hand.sch (KiCad schematic (older format))
At the start: 8 parts

Commit message: シート分けと移動
Parts:
- gave numbers to parts that had none: 8
Other:
- note added: "Etc."
Changed lines of the file:
@@
 $Descr A4 11693 8268
 encoding utf-8
-Sheet 4 4
+Sheet 4 6
 Title ""
 Date ""
@@
 $EndDescr
 $Comp
-L CONN_01X02 P?
+L CONN_01X02 P2
 U 1 1 593BE59D
 P 3800 3600
-F 0 "P?" H 3800 3750 50  0000 C CNN
+F 0 "P2" H 3800 3750 50  0000 C CNN
 F 1 "CW" V 3900 3600 50  0000 C CNN
 F 2 "" H 3800 3600 50  0000 C CNN
@@
 Connection ~ 4050 3550
 $Comp
-L +3.3V #PWR?
+L +3.3V #PWR026
 U 1 1 593BE5A9
 P 4050 3100
-F 0 "#PWR?" H 4050 2950 50  0001 C CNN
+F 0 "#PWR026" H 4050 2950 50  0001 C CNN
 F 1 "+3.3V" H 4050 3240 50  0000 C CNN
 F 2 "" H 4050 3100 50  0000 C CNN
@@
 $EndComp
 $Comp
-L R R?
+L R R6
 U 1 1 593BE5AF
 P 4050 3300
-F 0 "R?" V 4130 3300 50  0000 C CNN
+F 0 "R6" V 4130 3300 50  0000 C CNN
 F 1 "10k" V 4050 3300 50  0000 C CNN
 F 2 "" V 3980 3300 50  0000 C CNN
@@
 	4050 3150 4050 3100
 $Comp
-L GND #PWR?
+L GND #PWR027
 U 1 1 593BE5B7
 P 4050 3750
-F 0 "#PWR?" H 4050 3500 50  0001 C CNN
+F 0 "#PWR027" H 4050 3500 50  0001 C CNN
 F 1 "GND" H 4050 3600 50  0000 C CNN
 F 2 "" H 4050 3750 50  0000 C CNN
@@
 $EndComp
 $Comp
-L CONN_01X02 P?
+L CONN_01X02 P4
 U 1 1 593BE5BE
 P 4650 3600
-F 0 "P?" H 4650 3750 50  0000 C CNN
+F 0 "P4" H 4650 3750 50  0000 C CNN
 F 1 "CCW" V 4750 3600 50  0000 C CNN
 F 2 "" H 4650 3600 50  0000 C CNN
@@
 Connection ~ 4900 3550
 $Comp
-L +3.3V #PWR?
+L +3.3V #PWR028
 U 1 1 593BE5CA
 P 4900 3100
-F 0 "#PWR?" H 4900 2950 50  0001 C CNN
+F 0 "#PWR028" H 4900 2950 50  0001 C CNN
 F 1 "+3.3V" H 4900 3240 50  0000 C CNN
 F 2 "" H 4900 3100 50  0000 C CNN
@@
 $EndComp
 $Comp
-L R R?
+L R R8
 U 1 1 593BE5D0
 P 4900 3300
-F 0 "R?" V 4980 3300 50  0000 C CNN
+F 0 "R8" V 4980 3300 50  0000 C CNN
 F 1 "10k" V 4900 3300 50  0000 C CNN
 F 2 "" V 4830 3300 50  0000 C CNN
@@
 	4900 3150 4900 3100
 $Comp
-L GND #PWR?
+L GND #PWR029
 U 1 1 593BE5D8
 P 4900 3750
-F 0 "#PWR?" H 4900 3500 50  0001 C CNN
+F 0 "#PWR029" H 4900 3500 50  0001 C CNN
 F 1 "GND" H 4900 3600 50  0000 C CNN
 F 2 "" H 4900 3750 50  0000 C CNN
@@
 $EndComp
 $Comp
-L CONN_01X02 P?
+L CONN_01X02 P1
 U 1 1 593BE5DF
 P 3700 5150
-F 0 "P?" H 3700 5300 50  0000 C CNN
+F 0 "P1" H 3700 5300 50  0000 C CNN
 F 1 "Wall" V 3800 5150 50  0000 C CNN
 F 2 "" H 3700 5150 50  0000 C CNN
@@
 Connection ~ 3950 5100
 $Comp
-L +3.3V #PWR?
+L +3.3V #PWR030
 U 1 1 593BE5EB
 P 3950 4650
-F 0 "#PWR?" H 3950 4500 50  0001 C CNN
+F 0 "#PWR030" H 3950 4500 50  0001 C CNN
 F 1 "+3.3V" H 3950 4790 50  0000 C CNN
 F 2 "" H 3950 4650 50  0000 C CNN
@@
 $EndComp
 $Comp
-L R R?
+L R R5
 U 1 1 593BE5F1
 P 3950 4850
-F 0 "R?" V 4030 4850 50  0000 C CNN
+F 0 "R5" V 4030 4850 50  0000 C CNN
 F 1 "10k" V 3950 4850 50  0000 C CNN
 F 2 "" V 3880 4850 50  0000 C CNN
@@
 	3950 4700 3950 4650
 $Comp
-L GND #PWR?
+L GND #PWR031
 U 1 1 593BE5F9
 P 3950 5300
-F 0 "#PWR?" H 3950 5050 50  0001 C CNN
+F 0 "#PWR031" H 3950 5050 50  0001 C CNN
 F 1 "GND" H 3950 5150 50  0000 C CNN
 F 2 "" H 3950 5300 50  0000 C CNN
@@
 $EndComp
 $Comp
-L CONN_01X02 P?
+L CONN_01X02 P3
 U 1 1 593BE601
 P 4600 5150
-F 0 "P?" H 4600 5300 50  0000 C CNN
+F 0 "P3" H 4600 5300 50  0000 C CNN
 F 1 "Enable" V 4700 5150 50  0000 C CNN
 F 2 "" H 4600 5150 50  0000 C CNN
@@
 Connection ~ 4850 5100
 $Comp
-L +3.3V #PWR?
+L +3.3V #PWR032
 U 1 1 593BE60D
 P 4850 4650
-F 0 "#PWR?" H 4850 4500 50  0001 C CNN
+F 0 "#PWR032" H 4850 4500 50  0001 C CNN
 F 1 "+3.3V" H 4850 4790 50  0000 C CNN
 F 2 "" H 4850 4650 50  0000 C CNN
@@
 $EndComp
 $Comp
-L R R?
+L R R7
 U 1 1 593BE613
 P 4850 4850
-F 0 "R?" V 4930 4850 50  0000 C CNN
+F 0 "R7" V 4930 4850 50  0000 C CNN
 F 1 "10k" V 4850 4850 50  0000 C CNN
 F 2 "" V 4780 4850 50  0000 C CNN
@@
 	4850 4700 4850 4650
 $Comp
-L GND #PWR?
+L GND #PWR033
 U 1 1 593BE61B
 P 4850 5300
-F 0 "#PWR?" H 4850 5050 50  0001 C CNN
+F 0 "#PWR033" H 4850 5050 50  0001 C CNN
 F 1 "GND" H 4850 5150 50  0000 C CNN
 F 2 "" H 4850 5300 50  0000 C CNN
@@
 Text HLabel 5000 5100 2    60   Output ~ 0
 Enable
+Text Notes 5200 5650 0    60   ~ 0
+Etc.
 $EndSCHEMATC
