File: Circuit/Left_Hand.sch (KiCad schematic (older format))
At the start: 8 parts, among them P1 Wall, P2 CW, P3 Enable, P4 CCW

Commit message: 特になし
Parts:
- P1, P2, P3, P4: footprint (none) -> YASU:XA_2Pin
- R5, R6, R7, R8: footprint (none) -> Resistors_SMD:R_0603_HandSoldering
Changed lines of the file:
@@
 LIBS:contrib
 LIBS:valves
+LIBS:YASU
 LIBS:device
 LIBS:rhand_controller-cache
@@
 F 0 "P2" H 3800 3750 50  0000 C CNN
 F 1 "CW" V 3900 3600 50  0000 C CNN
-F 2 "" H 3800 3600 50  0000 C CNN
+F 2 "YASU:XA_2Pin" H 3800 3600 50  0001 C CNN
 F 3 "" H 3800 3600 50  0000 C CNN
 	1    3800 3600
@@
 F 0 "R6" V 4130 3300 50  0000 C CNN
 F 1 "10k" V 4050 3300 50  0000 C CNN
-F 2 "" V 3980 3300 50  0000 C CNN
+F 2 "Resistors_SMD:R_0603_HandSoldering" V 3980 3300 50  0001 C CNN
 F 3 "" H 4050 3300 50  0000 C CNN
 	1    4050 3300
@@
 F 0 "P4" H 4650 3750 50  0000 C CNN
 F 1 "CCW" V 4750 3600 50  0000 C CNN
-F 2 "" H 4650 3600 50  0000 C CNN
+F 2 "YASU:XA_2Pin" H 4650 3600 50  0001 C CNN
 F 3 "" H 4650 3600 50  0000 C CNN
 	1    4650 3600
@@
 F 0 "R8" V 4980 3300 50  0000 C CNN
 F 1 "10k" V 4900 3300 50  0000 C CNN
-F 2 "" V 4830 3300 50  0000 C CNN
+F 2 "Resistors_SMD:R_0603_HandSoldering" V 4830 3300 50  0001 C CNN
 F 3 "" H 4900 3300 50  0000 C CNN
 	1    4900 3300
@@
 F 0 "P1" H 3700 5300 50  0000 C CNN
 F 1 "Wall" V 3800 5150 50  0000 C CNN
-F 2 "" H 3700 5150 50  0000 C CNN
+F 2 "YASU:XA_2Pin" H 3700 5150 50  0001 C CNN
 F 3 "" H 3700 5150 50  0000 C CNN
 	1    3700 5150
@@
 F 0 "R5" V 4030 4850 50  0000 C CNN
 F 1 "10k" V 3950 4850 50  0000 C CNN
-F 2 "" V 3880 4850 50  0000 C CNN
+F 2 "Resistors_SMD:R_0603_HandSoldering" V 3880 4850 50  0001 C CNN
 F 3 "" H 3950 4850 50  0000 C CNN
 	1    3950 4850
@@
 F 0 "P3" H 4600 5300 50  0000 C CNN
 F 1 "Enable" V 4700 5150 50  0000 C CNN
-F 2 "" H 4600 5150 50  0000 C CNN
+F 2 "YASU:XA_2Pin" H 4600 5150 50  0001 C CNN
 F 3 "" H 4600 5150 50  0000 C CNN
 	1    4600 5150
@@
 F 0 "R7" V 4930 4850 50  0000 C CNN
 F 1 "10k" V 4850 4850 50  0000 C CNN
-F 2 "" V 4780 4850 50  0000 C CNN
+F 2 "Resistors_SMD:R_0603_HandSoldering" V 4780 4850 50  0001 C CNN
 F 3 "" H 4850 4850 50  0000 C CNN
 	1    4850 4850
