File: Circuit/ST-LINK.sch (KiCad schematic (older format))
At the start: 1 part, among them P17 CONN_01X06

Commit message: シート分けと移動
Parts:
- added R3: 1k, Resistors_SMD:R_0603_HandSoldering, symbol R
Connections:
- net NRST: now also R3.2
- new net +3V3: R3.1
Changed lines of the file:
@@
 $Descr A4 11693 8268
 encoding utf-8
-Sheet 2 4
+Sheet 2 6
 Title ""
 Date ""
@@
 	3500 2800 3500 3200
 Wire Wire Line
-	3600 3000 3400 3000
-Wire Wire Line
 	3600 3100 3400 3100
 $Comp
-L GND #PWR047
+L GND #PWR022
 U 1 1 58DA69EB
 P 3500 3200
-F 0 "#PWR047" H 3500 2950 50  0001 C CNN
+F 0 "#PWR022" H 3500 2950 50  0001 C CNN
 F 1 "GND" H 3500 3050 50  0000 C CNN
 F 2 "" H 3500 3200 50  0000 C CNN
@@
 Text HLabel 3400 2900 0    60   Output ~ 0
 SWDIO
-Text HLabel 3400 3000 0    60   Output ~ 0
+Text HLabel 2700 3000 0    60   Output ~ 0
 NRST
 Text HLabel 3400 3100 0    60   Output ~ 0
 SWO
+$Comp
+L R R3
+U 1 1 593DD523
+P 2850 2800
+F 0 "R3" V 2930 2800 50  0000 C CNN
+F 1 "1k" V 2850 2800 50  0000 C CNN
+F 2 "Resistors_SMD:R_0603_HandSoldering" V 2780 2800 50  0001 C CNN
+F 3 "" H 2850 2800 50  0000 C CNN
+	1    2850 2800
+	1    0    0    -1
+$EndComp
+$Comp
+L +3.3V #PWR023
+U 1 1 593DD52A
+P 2850 2500
+F 0 "#PWR023" H 2850 2350 50  0001 C CNN
+F 1 "+3.3V" H 2850 2640 50  0000 C CNN
+F 2 "" H 2850 2500 50  0000 C CNN
+F 3 "" H 2850 2500 50  0000 C CNN
+	1    2850 2500
+	1    0    0    -1
+$EndComp
+Wire Wire Line
+	2700 3000 3600 3000
+Wire Wire Line
+	2850 2950 2850 3000
+Wire Wire Line
+	2850 2500 2850 2650
+Connection ~ 2850 3000
 $EndSCHEMATC
