File: Circuit/rhand_controller.sch (KiCad schematic (older format))
At the start: 16 parts

Commit message: 部品の割り付け
Parts:
- BT1: renamed from BT?; value Battery -> LiPo
- C1, C2: renamed from C?; value C -> 0.1u; footprint (none) -> Capacitors_SMD:C_0805_HandSoldering
- P2: renamed from P?; value U_ADC -> LU_ADC
- P4: renamed from P?; value V_ADC -> LV_ADC
- P6: renamed from P?; value W_ADC -> LW_ADC
- R1: renamed from R?; value R -> 1k; footprint (none) -> Resistors_SMD:R_0603_HandSoldering
- R2, R3: renamed from R?; footprint (none) -> Resistors_SMD:R_0603_HandSoldering
- gave numbers to parts that had none: 7
Changed lines of the file:
@@
 $EndSheet
 $Comp
-L STM32F042 U?
+L STM32F042 U1
 U 1 1 5936B864
 P 4800 5200
-F 0 "U?" H 5400 5100 60  0000 C CNN
+F 0 "U1" H 5400 5100 60  0000 C CNN
 F 1 "STM32F042" H 5400 5250 60  0000 C CNN
-F 2 "" H 5350 5100 60  0000 C CNN
+F 2 "" H 5350 5100 60  0001 C CNN
 F 3 "" H 5350 5100 60  0000 C CNN
 	1    4800 5200
@@
 $EndComp
 $Comp
-L BLUETOOTH P?
+L BLUETOOTH P7
 U 1 1 5936B91F
 P 9200 1500
-F 0 "P?" H 9200 1900 60  0000 C CNN
+F 0 "P7" H 9200 1900 60  0000 C CNN
 F 1 "BLUETOOTH" H 9200 1300 60  0000 C CNN
-F 2 "" H 9200 1500 60  0000 C CNN
+F 2 "" H 9200 1500 60  0001 C CNN
 F 3 "" H 9200 1500 60  0000 C CNN
 	1    9200 1500
@@
 $EndComp
 $Comp
-L C C?
+L C C1
 U 1 1 5936C50E
 P 5250 3400
-F 0 "C?" H 5275 3500 50  0000 L CNN
-F 1 "C" H 5275 3300 50  0000 L CNN
-F 2 "" H 5288 3250 50  0000 C CNN
+F 0 "C1" H 5275 3500 50  0000 L CNN
+F 1 "0.1u" H 5275 3300 50  0000 L CNN
+F 2 "Capacitors_SMD:C_0805_HandSoldering" H 5288 3250 50  0001 C CNN
 F 3 "" H 5250 3400 50  0000 C CNN
 	1    5250 3400
@@
 SWO
 $Comp
-L R R?
+L R R3
 U 1 1 5936DE36
 P 9750 4950
-F 0 "R?" V 9830 4950 50  0000 C CNN
+F 0 "R3" V 9830 4950 50  0000 C CNN
 F 1 "1k" V 9750 4950 50  0000 C CNN
-F 2 "" V 9680 4950 50  0000 C CNN
+F 2 "Resistors_SMD:R_0603_HandSoldering" V 9680 4950 50  0001 C CNN
 F 3 "" H 9750 4950 50  0000 C CNN
 	1    9750 4950
@@
 $EndComp
 $Comp
-L R R?
+L R R2
 U 1 1 5936E3FC
 P 8500 4700
-F 0 "R?" V 8580 4700 50  0000 C CNN
+F 0 "R2" V 8580 4700 50  0000 C CNN
 F 1 "10k" V 8500 4700 50  0000 C CNN
-F 2 "" V 8430 4700 50  0000 C CNN
+F 2 "Resistors_SMD:R_0603_HandSoldering" V 8430 4700 50  0001 C CNN
 F 3 "" H 8500 4700 50  0000 C CNN
 	1    8500 4700
@@
 $EndComp
 $Comp
-L CONN_01X03 P?
+L CONN_01X03 P3
 U 1 1 593711C9
 P 2350 1450
-F 0 "P?" H 2350 1650 50  0000 C CNN
+F 0 "P3" H 2350 1650 50  0000 C CNN
 F 1 "RV_ADC" V 2450 1450 50  0000 C CNN
-F 2 "" H 2350 1450 50  0000 C CNN
+F 2 "" H 2350 1450 50  0001 C CNN
 F 3 "" H 2350 1450 50  0000 C CNN
 	1    2350 1450
@@
 $EndComp
 $Comp
-L CONN_01X03 P?
+L CONN_01X03 P5
 U 1 1 59371792
 P 3100 1450
-F 0 "P?" H 3100 1650 50  0000 C CNN
+F 0 "P5" H 3100 1650 50  0000 C CNN
 F 1 "RW_ADC" V 3200 1450 50  0000 C CNN
-F 2 "" H 3100 1450 50  0000 C CNN
+F 2 "" H 3100 1450 50  0001 C CNN
 F 3 "" H 3100 1450 50  0000 C CNN
 	1    3100 1450
@@
 $EndComp
 $Comp
-L CONN_01X03 P?
+L CONN_01X03 P1
 U 1 1 593717F9
 P 1600 1450
-F 0 "P?" H 1600 1650 50  0000 C CNN
+F 0 "P1" H 1600 1650 50  0000 C CNN
 F 1 "RU_ADC" V 1700 1450 50  0000 C CNN
-F 2 "" H 1600 1450 50  0000 C CNN
+F 2 "" H 1600 1450 50  0001 C CNN
 F 3 "" H 1600 1450 50  0000 C CNN
 	1    1600 1450
@@
 RSW_B3
 $Comp
-L C C?
+L C C2
 U 1 1 5937C110
 P 9850 1750
-F 0 "C?" H 9875 1850 50  0000 L CNN
-F 1 "C" H 9875 1650 50  0000 L CNN
-F 2 "" H 9888 1600 50  0000 C CNN
+F 0 "C2" H 9875 1850 50  0000 L CNN
+F 1 "0.1u" H 9875 1650 50  0000 L CNN
+F 2 "Capacitors_SMD:C_0805_HandSoldering" H 9888 1600 50  0001 C CNN
 F 3 "" H 9850 1750 50  0000 C CNN
 	1    9850 1750
@@
 $EndComp
 $Comp
-L CONN_01X03 P?
+L CONN_01X03 P4
 U 1 1 59376C0C
 P 2350 2200
-F 0 "P?" H 2350 2400 50  0000 C CNN
-F 1 "V_ADC" V 2450 2200 50  0000 C CNN
-F 2 "" H 2350 2200 50  0000 C CNN
+F 0 "P4" H 2350 2400 50  0000 C CNN
+F 1 "LV_ADC" V 2450 2200 50  0000 C CNN
+F 2 "" H 2350 2200 50  0001 C CNN
 F 3 "" H 2350 2200 50  0000 C CNN
 	1    2350 2200
@@
 $EndComp
 $Comp
-L CONN_01X03 P?
+L CONN_01X03 P6
 U 1 1 59376C12
 P 3100 2200
-F 0 "P?" H 3100 2400 50  0000 C CNN
-F 1 "W_ADC" V 3200 2200 50  0000 C CNN
-F 2 "" H 3100 2200 50  0000 C CNN
+F 0 "P6" H 3100 2400 50  0000 C CNN
+F 1 "LW_ADC" V 3200 2200 50  0000 C CNN
+F 2 "" H 3100 2200 50  0001 C CNN
 F 3 "" H 3100 2200 50  0000 C CNN
 	1    3100 2200
@@
 $EndComp
 $Comp
-L CONN_01X03 P?
+L CONN_01X03 P2
 U 1 1 59376C18
 P 1600 2200
-F 0 "P?" H 1600 2400 50  0000 C CNN
-F 1 "U_ADC" V 1700 2200 50  0000 C CNN
-F 2 "" H 1600 2200 50  0000 C CNN
+F 0 "P2" H 1600 2400 50  0000 C CNN
+F 1 "LU_ADC" V 1700 2200 50  0000 C CNN
+F 2 "" H 1600 2200 50  0001 C CNN
 F 3 "" H 1600 2200 50  0000 C CNN
 	1    1600 2200
@@
 $EndComp
 $Comp
-L GND #PWR?
+L GND #PWR015
 U 1 1 59376C1E
 P 1800 2350
-F 0 "#PWR?" H 1800 2100 50  0001 C CNN
+F 0 "#PWR015" H 1800 2100 50  0001 C CNN
 F 1 "GND" H 1800 2200 50  0000 C CNN
 F 2 "" H 1800 2350 50  0000 C CNN
@@
 $EndComp
 $Comp
-L GND #PWR?
+L GND #PWR016
 U 1 1 59376C24
 P 2550 2350
-F 0 "#PWR?" H 2550 2100 50  0001 C CNN
+F 0 "#PWR016" H 2550 2100 50  0001 C CNN
 F 1 "GND" H 2550 2200 50  0000 C CNN
 F 2 "" H 2550 2350 50  0000 C CNN
@@
 $EndComp
 $Comp
-L GND #PWR?
+L GND #PWR017
 U 1 1 59376C2A
 P 3300 2350
-F 0 "#PWR?" H 3300 2100 50  0001 C CNN
+F 0 "#PWR017" H 3300 2100 50  0001 C CNN
 F 1 "GND" H 3300 2200 50  0000 C CNN
 F 2 "" H 3300 2350 50  0000 C CNN
@@
 $EndComp
 $Comp
-L +3.3V #PWR?
+L +3.3V #PWR018
 U 1 1 59376C33
 P 3300 2050
-F 0 "#PWR?" H 3300 1900 50  0001 C CNN
+F 0 "#PWR018" H 3300 1900 50  0001 C CNN
 F 1 "+3.3V" H 3300 2190 50  0000 C CNN
 F 2 "" H 3300 2050 50  0000 C CNN
@@
 $EndComp
 $Comp
-L +3.3V #PWR?
+L +3.3V #PWR019
 U 1 1 59376C39
 P 2550 2050
-F 0 "#PWR?" H 2550 1900 50  0001 C CNN
+F 0 "#PWR019" H 2550 1900 50  0001 C CNN
 F 1 "+3.3V" H 2550 2190 50  0000 C CNN
 F 2 "" H 2550 2050 50  0000 C CNN
@@
 $EndComp
 $Comp
-L +3.3V #PWR?
+L +3.3V #PWR020
 U 1 1 59376C3F
 P 1800 2050
-F 0 "#PWR?" H 1800 1900 50  0001 C CNN
+F 0 "#PWR020" H 1800 1900 50  0001 C CNN
 F 1 "+3.3V" H 1800 2190 50  0000 C CNN
 F 2 "" H 1800 2050 50  0000 C CNN
@@
 	1100 4700 1450 4700
 $Comp
-L Battery BT?
+L Battery BT1
 U 1 1 59383F89
 P 10500 2650
-F 0 "BT?" H 10600 2750 50  0000 L CNN
-F 1 "Battery" H 10600 2650 50  0000 L CNN
+F 0 "BT1" H 10600 2750 50  0000 L CNN
+F 1 "LiPo" H 10600 2650 50  0000 L CNN
 F 2 "" V 10500 2710 50  0001 C CNN
 F 3 "" V 10500 2710 50  0001 C CNN
@@
 $EndComp
 $Comp
-L +7.4V #PWR?
+L +7.4V #PWR021
 U 1 1 59384263
 P 10500 2350
-F 0 "#PWR?" H 10500 2200 50  0001 C CNN
+F 0 "#PWR021" H 10500 2200 50  0001 C CNN
 F 1 "+7.4V" H 10500 2490 50  0000 C CNN
 F 2 "" H 10500 2350 50  0001 C CNN
@@
 	10500 2850 10500 2950
 $Comp
-L GND #PWR?
+L GND #PWR022
 U 1 1 593848DF
 P 10500 2950
-F 0 "#PWR?" H 10500 2700 50  0001 C CNN
+F 0 "#PWR022" H 10500 2700 50  0001 C CNN
 F 1 "GND" H 10500 2800 50  0000 C CNN
 F 2 "" H 10500 2950 50  0001 C CNN
@@
 $EndComp
 $Comp
-L PWR_FLAG #FLG?
+L PWR_FLAG #FLG023
 U 1 1 59384943
 P 10850 2350
-F 0 "#FLG?" H 10850 2425 50  0001 C CNN
+F 0 "#FLG023" H 10850 2425 50  0001 C CNN
 F 1 "PWR_FLAG" H 10850 2500 50  0000 C CNN
 F 2 "" H 10850 2350 50  0001 C CNN
@@
 Connection ~ 10500 2900
 $Comp
-L PWR_FLAG #FLG?
+L PWR_FLAG #FLG024
 U 1 1 59384B48
 P 10850 2950
-F 0 "#FLG?" H 10850 3025 50  0001 C CNN
+F 0 "#FLG024" H 10850 3025 50  0001 C CNN
 F 1 "PWR_FLAG" H 10850 3100 50  0000 C CNN
 F 2 "" H 10850 2950 50  0001 C CNN
@@
 $EndComp
 $Comp
-L +7.4V #PWR?
+L +7.4V #PWR025
 U 1 1 5938507B
 P 10100 5900
-F 0 "#PWR?" H 10100 5750 50  0001 C CNN
+F 0 "#PWR025" H 10100 5750 50  0001 C CNN
 F 1 "+7.4V" H 10100 6040 50  0000 C CNN
 F 2 "" H 10100 5900 50  0001 C CNN
@@
 $EndComp
 $Comp
-L IM315TX U?
+L IM315TX U2
 U 1 1 59389911
 P 6250 1500
-F 0 "U?" H 5900 2000 60  0000 C CNN
+F 0 "U2" H 5900 2000 60  0000 C CNN
 F 1 "IM315TX" H 6600 2000 60  0000 C CNN
 F 2 "" H 5825 1875 60  0001 C CNN
@@
 $EndComp
 $Comp
-L +3.3V #PWR?
+L +3.3V #PWR026
 U 1 1 5938AB88
 P 6250 800
-F 0 "#PWR?" H 6250 650 50  0001 C CNN
+F 0 "#PWR026" H 6250 650 50  0001 C CNN
 F 1 "+3.3V" H 6250 940 50  0000 C CNN
 F 2 "" H 6250 800 50  0000 C CNN
@@
 	6250 2150 6250 2200
 $Comp
-L GND #PWR?
+L GND #PWR027
 U 1 1 5938B2E2
 P 6250 2200
-F 0 "#PWR?" H 6250 1950 50  0001 C CNN
+F 0 "#PWR027" H 6250 1950 50  0001 C CNN
 F 1 "GND" H 6250 2050 50  0000 C CNN
 F 2 "" H 6250 2200 50  0000 C CNN
@@
 NoConn ~ 5500 1850
 $Comp
-L LED D?
+L LED D1
 U 1 1 5938D7FB
 P 7650 1750
-F 0 "D?" H 7650 1850 50  0000 C CNN
+F 0 "D1" H 7650 1850 50  0000 C CNN
 F 1 "LED" H 7650 1650 50  0000 C CNN
 F 2 "" H 7650 1750 50  0001 C CNN
@@
 	7650 1900 7650 2000
 $Comp
-L R R?
+L R R1
 U 1 1 5938D995
 P 7650 2150
-F 0 "R?" V 7730 2150 50  0000 C CNN
-F 1 "R" V 7650 2150 50  0000 C CNN
-F 2 "" V 7580 2150 50  0001 C CNN
+F 0 "R1" V 7730 2150 50  0000 C CNN
+F 1 "1k" V 7650 2150 50  0000 C CNN
+F 2 "Resistors_SMD:R_0603_HandSoldering" V 7580 2150 50  0001 C CNN
 F 3 "" H 7650 2150 50  0001 C CNN
 	1    7650 2150
@@
 	7650 2300 7650 2400
 $Comp
-L GND #PWR?
+L GND #PWR028
 U 1 1 5938DB33
 P 7650 2400
-F 0 "#PWR?" H 7650 2150 50  0001 C CNN
+F 0 "#PWR028" H 7650 2150 50  0001 C CNN
 F 1 "GND" H 7650 2250 50  0000 C CNN
 F 2 "" H 7650 2400 50  0001 C CNN
@@
 	7100 1200 7100 1150
 $Comp
-L +3.3V #PWR?
+L +3.3V #PWR029
 U 1 1 5938E5AC
 P 7100 1150
-F 0 "#PWR?" H 7100 1000 50  0001 C CNN
+F 0 "#PWR029" H 7100 1000 50  0001 C CNN
 F 1 "+3.3V" H 7100 1290 50  0000 C CNN
 F 2 "" H 7100 1150 50  0000 C CNN
@@
 	7450 1750 7000 1750
 $Comp
-L GND #PWR?
+L GND #PWR030
 U 1 1 5938FDF2
 P 7100 1350
-F 0 "#PWR?" H 7100 1100 50  0001 C CNN
+F 0 "#PWR030" H 7100 1100 50  0001 C CNN
 F 1 "GND" H 7100 1200 50  0000 C CNN
 F 2 "" H 7100 1350 50  0000 C CNN

Commit message: 機能の追加
Parts:
- added P?: RW_ADC, symbol CONN_01X03
- added P?: LW_ADC, symbol CONN_01X03
- added P?: CW, symbol CONN_01X02
- added P?: CCW, symbol CONN_01X02
- added P?: Wall, symbol CONN_01X02
- added P?: Enable, symbol CONN_01X02
- added R? (x8): 10k, symbol R
- added S?: SW_DIP_x4, symbol SW_DIP_x4
- added SW?: EmSW, symbol SW_PUSH
- added SW?: SWITCH_INV, symbol SWITCH_INV
Connections:
- net labels added: CCW, CW, DSW_B0, DSW_B1, DSW_B2, Enable, Joy_X, Joy_Y, Wall
- net labels removed: RSW_B0, RSW_B1, RSW_B2, RSW_B3
- wire segments 92 -> 141
- no-connect marks 11 -> 8
Other:
- moved on the sheet: BT1, C1, C2, D1, P1, P2, P3, P4, P5, P6, P7, R1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

Commit message: 何を変えたか忘れたけど更新
Parts:
- gave numbers to parts that had none: 17
Connections:
- net +3V3: now also S1.5; no longer S1.8
- net DSW_B0: now also S1.2; no longer S1.1
- net DSW_B1: now also S1.3; no longer S1.2
- net DSW_B2: now also S1.4; no longer S1.3
- net GND: no longer BT1.2
- net at BT1.1: no longer SW2.1
Other:
- moved on the sheet: BT1, R10, R11, R9

Commit message: シートわけ
Parts:
- removed P10: CCW, symbol CONN_01X02
- removed P12: Wall, symbol CONN_01X02
- removed P13: Enable, symbol CONN_01X02
- removed P8: CW, symbol CONN_01X02
- removed R5, R6, R7, R8: 10k, symbol R
Changed lines of the file:
@@
 $Descr A4 11693 8268
 encoding utf-8
-Sheet 1 3
+Sheet 1 4
 Title ""
 Date ""
@@
 $EndComp
 $Comp
-L CONN_01X02 P8
-U 1 1 59397274
-P 1000 3800
-F 0 "P8" H 1000 3950 50  0000 C CNN
-F 1 "CW" V 1100 3800 50  0000 C CNN
-F 2 "" H 1000 3800 50  0000 C CNN
-F 3 "" H 1000 3800 50  0000 C CNN
-	1    1000 3800
-	-1   0    0    1
-$EndComp
-$Comp
 L SW_DIP_x4 S1
 U 1 1 593A8DBA
@@
 	1    0    0    -1
 $EndComp
-Wire Wire Line
-	1200 3750 1500 3750
-Wire Wire Line
-	1250 3650 1250 3750
-Wire Wire Line
-	1200 3850 1250 3850
-Wire Wire Line
-	1250 3850 1250 3950
-Connection ~ 1250 3750
-$Comp
-L +3.3V #PWR039
-U 1 1 593B0066
-P 1250 3300
-F 0 "#PWR039" H 1250 3150 50  0001 C CNN
-F 1 "+3.3V" H 1250 3440 50  0000 C CNN
-F 2 "" H 1250 3300 50  0000 C CNN
-F 3 "" H 1250 3300 50  0000 C CNN
-	1    1250 3300
-	1    0    0    -1
-$EndComp
-$Comp
-L R R5
-U 1 1 593B02B9
-P 1250 3500
-F 0 "R5" V 1330 3500 50  0000 C CNN
-F 1 "10k" V 1250 3500 50  0000 C CNN
-F 2 "" V 1180 3500 50  0000 C CNN
-F 3 "" H 1250 3500 50  0000 C CNN
-	1    1250 3500
-	1    0    0    -1
-$EndComp
-Wire Wire Line
-	1250 3350 1250 3300
-$Comp
-L GND #PWR040
-U 1 1 593B0436
-P 1250 3950
-F 0 "#PWR040" H 1250 3700 50  0001 C CNN
-F 1 "GND" H 1250 3800 50  0000 C CNN
-F 2 "" H 1250 3950 50  0000 C CNN
-F 3 "" H 1250 3950 50  0000 C CNN
-	1    1250 3950
-	1    0    0    -1
-$EndComp
-Text Label 1500 3750 2    60   ~ 0
-CW
-$Comp
-L CONN_01X02 P10
-U 1 1 593B0FF5
-P 1800 3800
-F 0 "P10" H 1800 3950 50  0000 C CNN
-F 1 "CCW" V 1900 3800 50  0000 C CNN
-F 2 "" H 1800 3800 50  0000 C CNN
-F 3 "" H 1800 3800 50  0000 C CNN
-	1    1800 3800
-	-1   0    0    1
-$EndComp
-Wire Wire Line
-	2000 3750 2350 3750
-Wire Wire Line
-	2050 3650 2050 3750
-Wire Wire Line
-	2000 3850 2050 3850
-Wire Wire Line
-	2050 3850 2050 3950
-Connection ~ 2050 3750
-$Comp
-L +3.3V #PWR041
-U 1 1 593B1000
-P 2050 3300
-F 0 "#PWR041" H 2050 3150 50  0001 C CNN
-F 1 "+3.3V" H 2050 3440 50  0000 C CNN
-F 2 "" H 2050 3300 50  0000 C CNN
-F 3 "" H 2050 3300 50  0000 C CNN
-	1    2050 3300
-	1    0    0    -1
-$EndComp
-$Comp
-L R R6
-U 1 1 593B1006
-P 2050 3500
-F 0 "R6" V 2130 3500 50  0000 C CNN
-F 1 "10k" V 2050 3500 50  0000 C CNN
-F 2 "" V 1980 3500 50  0000 C CNN
-F 3 "" H 2050 3500 50  0000 C CNN
-	1    2050 3500
-	1    0    0    -1
-$EndComp
-Wire Wire Line
-	2050 3350 2050 3300
-$Comp
-L GND #PWR042
-U 1 1 593B100D
-P 2050 3950
-F 0 "#PWR042" H 2050 3700 50  0001 C CNN
-F 1 "GND" H 2050 3800 50  0000 C CNN
-F 2 "" H 2050 3950 50  0000 C CNN
-F 3 "" H 2050 3950 50  0000 C CNN
-	1    2050 3950
-	1    0    0    -1
-$EndComp
-Text Label 2350 3750 2    60   ~ 0
-CCW
 Text Label 1450 5550 0    60   ~ 0
 CW
@@
 Wire Wire Line
 	4850 2150 4850 2100
-$Comp
-L CONN_01X02 P12
-U 1 1 593C2B7D
-P 2600 3800
-F 0 "P12" H 2600 3950 50  0000 C CNN
-F 1 "Wall" V 2700 3800 50  0000 C CNN
-F 2 "" H 2600 3800 50  0000 C CNN
-F 3 "" H 2600 3800 50  0000 C CNN
-	1    2600 3800
-	-1   0    0    1
-$EndComp
-Wire Wire Line
-	2800 3750 3150 3750
-Wire Wire Line
-	2850 3650 2850 3750
-Wire Wire Line
-	2800 3850 2850 3850
-Wire Wire Line
-	2850 3850 2850 3950
-Connection ~ 2850 3750
-$Comp
-L +3.3V #PWR043
-U 1 1 593C2B89
-P 2850 3300
-F 0 "#PWR043" H 2850 3150 50  0001 C CNN
-F 1 "+3.3V" H 2850 3440 50  0000 C CNN
-F 2 "" H 2850 3300 50  0000 C CNN
-F 3 "" H 2850 3300 50  0000 C CNN
-	1    2850 3300
-	1    0    0    -1
-$EndComp
-$Comp
-L R R7
-U 1 1 593C2B8F
-P 2850 3500
-F 0 "R7" V 2930 3500 50  0000 C CNN
-F 1 "10k" V 2850 3500 50  0000 C CNN
-F 2 "" V 2780 3500 50  0000 C CNN
-F 3 "" H 2850 3500 50  0000 C CNN
-	1    2850 3500
-	1    0    0    -1
-$EndComp
-Wire Wire Line
-	2850 3350 2850 3300
-$Comp
-L GND #PWR044
-U 1 1 593C2B96
-P 2850 3950
-F 0 "#PWR044" H 2850 3700 50  0001 C CNN
-F 1 "GND" H 2850 3800 50  0000 C CNN
-F 2 "" H 2850 3950 50  0000 C CNN
-F 3 "" H 2850 3950 50  0000 C CNN
-	1    2850 3950
-	1    0    0    -1
-$EndComp
-Text Label 3150 3750 2    60   ~ 0
-Wall
 Text Label 8850 5800 2    60   ~ 0
 Wall
@@
 Text Label 8850 5900 2    60   ~ 0
 Enable
-Text Label 4050 3750 2    60   ~ 0
-Enable
-$Comp
-L CONN_01X02 P13
-U 1 1 593C433B
-P 3400 3800
-F 0 "P13" H 3400 3950 50  0000 C CNN
-F 1 "Enable" V 3500 3800 50  0000 C CNN
-F 2 "" H 3400 3800 50  0000 C CNN
-F 3 "" H 3400 3800 50  0000 C CNN
-	1    3400 3800
-	-1   0    0    1
-$EndComp
-Wire Wire Line
-	3600 3750 4050 3750
-Wire Wire Line
-	3650 3650 3650 3750
-Wire Wire Line
-	3600 3850 3650 3850
-Wire Wire Line
-	3650 3850 3650 3950
-Connection ~ 3650 3750
-$Comp
-L +3.3V #PWR045
-U 1 1 593C4346
-P 3650 3300
-F 0 "#PWR045" H 3650 3150 50  0001 C CNN
-F 1 "+3.3V" H 3650 3440 50  0000 C CNN
-F 2 "" H 3650 3300 50  0000 C CNN
-F 3 "" H 3650 3300 50  0000 C CNN
-	1    3650 3300
-	1    0    0    -1
-$EndComp
-$Comp
-L R R8
-U 1 1 593C434C
-P 3650 3500
-F 0 "R8" V 3730 3500 50  0000 C CNN
-F 1 "10k" V 3650 3500 50  0000 C CNN
-F 2 "" V 3580 3500 50  0000 C CNN
-F 3 "" H 3650 3500 50  0000 C CNN
-	1    3650 3500
-	1    0    0    -1
-$EndComp
-Wire Wire Line
-	3650 3350 3650 3300
-$Comp
-L GND #PWR046
-U 1 1 593C4353
-P 3650 3950
-F 0 "#PWR046" H 3650 3700 50  0001 C CNN
-F 1 "GND" H 3650 3800 50  0000 C CNN
-F 2 "" H 3650 3950 50  0000 C CNN
-F 3 "" H 3650 3950 50  0000 C CNN
-	1    3650 3950
-	1    0    0    -1
-$EndComp
 Wire Wire Line
 	4850 2550 4850 2650
@@
 	4850 2600 5200 2600
 Connection ~ 4850 2600
+$Sheet
+S 1950 3450 700  300
+U 593BDA75
+F0 "DIO" 60
+F1 "Digital_input.sch" 60
+$EndSheet
 $EndSCHEMATC

Commit message: シート分けと移動
Parts:
- removed P1: RU_ADC, symbol CONN_01X03
- removed P11, P5: RW_ADC, symbol CONN_01X03
- removed P2: LU_ADC, symbol CONN_01X03
- removed P3: RV_ADC, symbol CONN_01X03
- removed P4: LV_ADC, symbol CONN_01X03
- removed P6, P9: LW_ADC, symbol CONN_01X03
- removed R3: 1k, Resistors_SMD:R_0603_HandSoldering, symbol R
Connections:
- net +3V3: now also C2.2; no longer C2.1
- net GND: now also BT1.2, C2.1; no longer C2.2
- net at BT1.1: now also SW2.1
- net at D1.1 (K): now also R1.1
Other:
- note added: "Communication module"
- moved on the sheet: BT1, C1, C2, D1, P7, R1, R10, R11, R2, R4, R9, S1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
