File: Circuit/Arms.sch (KiCad schematic (older format))
At the start: 6 parts, among them P10 LW_ADC, P11 RU_ADC, P12 RV_ADC, P13 RW_ADC, P8 LU_ADC, P9 LV_ADC

Commit message: 特になし
Parts:
- P10, P11, P12, P13, P8, P9: footprint (none) -> YASU:XA_3Pin
Changed lines of the file:
@@
 LIBS:contrib
 LIBS:valves
+LIBS:YASU
 LIBS:device
 LIBS:rhand_controller-cache
@@
 F 0 "P12" H 4850 4650 50  0000 C CNN
 F 1 "RV_ADC" V 4950 4450 50  0000 C CNN
-F 2 "" H 4850 4450 50  0001 C CNN
+F 2 "YASU:XA_3Pin" H 4850 4450 50  0001 C CNN
 F 3 "" H 4850 4450 50  0000 C CNN
 	1    4850 4450
@@
 F 0 "P13" H 4850 5400 50  0000 C CNN
 F 1 "RW_ADC" V 4950 5200 50  0000 C CNN
-F 2 "" H 4850 5200 50  0001 C CNN
+F 2 "YASU:XA_3Pin" H 4850 5200 50  0001 C CNN
 F 3 "" H 4850 5200 50  0000 C CNN
 	1    4850 5200
@@
 F 0 "P11" H 4850 3900 50  0000 C CNN
 F 1 "RU_ADC" V 4950 3700 50  0000 C CNN
-F 2 "" H 4850 3700 50  0001 C CNN
+F 2 "YASU:XA_3Pin" H 4850 3700 50  0001 C CNN
 F 3 "" H 4850 3700 50  0000 C CNN
 	1    4850 3700
@@
 F 0 "P9" H 3600 4650 50  0000 C CNN
 F 1 "LV_ADC" V 3700 4450 50  0000 C CNN
-F 2 "" H 3600 4450 50  0001 C CNN
+F 2 "YASU:XA_3Pin" H 3600 4450 50  0001 C CNN
 F 3 "" H 3600 4450 50  0000 C CNN
 	1    3600 4450
@@
 F 0 "P10" H 3600 5400 50  0000 C CNN
 F 1 "LW_ADC" V 3700 5200 50  0000 C CNN
-F 2 "" H 3600 5200 50  0001 C CNN
+F 2 "YASU:XA_3Pin" H 3600 5200 50  0001 C CNN
 F 3 "" H 3600 5200 50  0000 C CNN
 	1    3600 5200
@@
 F 0 "P8" H 3600 3900 50  0000 C CNN
 F 1 "LU_ADC" V 3700 3700 50  0000 C CNN
-F 2 "" H 3600 3700 50  0001 C CNN
+F 2 "YASU:XA_3Pin" H 3600 3700 50  0001 C CNN
 F 3 "" H 3600 3700 50  0000 C CNN
 	1    3600 3700
