File: Circuit/Right_hand.sch (KiCad schematic (older format))
At the start: 2 parts, among them P5 LW_ADC, P6 RW_ADC

Commit message: 特になし
Parts:
- P5, P6: footprint (none) -> YASU:XA_3Pin
Changed lines of the file:
@@
 LIBS:contrib
 LIBS:valves
+LIBS:YASU
 LIBS:device
 LIBS:rhand_controller-cache
@@
 F 0 "P6" H 4400 4300 50  0000 C CNN
 F 1 "RW_ADC" V 4500 4100 50  0000 C CNN
-F 2 "" H 4400 4100 50  0001 C CNN
+F 2 "YASU:XA_3Pin" H 4400 4100 50  0001 C CNN
 F 3 "" H 4400 4100 50  0000 C CNN
 	1    4400 4100
@@
 F 0 "P5" H 4400 3550 50  0000 C CNN
 F 1 "LW_ADC" V 4500 3350 50  0000 C CNN
-F 2 "" H 4400 3350 50  0001 C CNN
+F 2 "YASU:XA_3Pin" H 4400 3350 50  0001 C CNN
 F 3 "" H 4400 3350 50  0000 C CNN
 	1    4400 3350
