File: Circuit/rhand_controller.kicad_pcb (KiCad board)
At the start: 2 copper layers, 100 x 100 mm, 39 parts, among them P1 BLUETOOTH, P10 LV_ADC, P11 LW_ADC, P12 RU_ADC, P13 RV_ADC, P14 RW_ADC, P2 CONN_01X06, P3 Wall, P4 CW, P5 Enable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

Commit message: 基板固定用の穴と三端子レギュレータ回りの配線の変更
Parts:
- added REF**: MountingHole_3.2mm_M3, Mounting_Holes:MountingHole_3.2mm_M3, F.Cu at (147.0, 73.0)
- added REF**: MountingHole_3.2mm_M3, Mounting_Holes:MountingHole_3.2mm_M3, F.Cu at (53.0, 73.0)
- added REF**: MountingHole_3.2mm_M3, Mounting_Holes:MountingHole_3.2mm_M3, F.Cu at (147.0, 167.0)
- added REF**: MountingHole_3.2mm_M3, Mounting_Holes:MountingHole_3.2mm_M3, F.Cu at (53.0, 167.0)
- moved P10 5.41 mm to (124.8, 161.0)
- moved P11 5.41 mm to (110.0, 161.0)
- moved P12 5.41 mm to (90.0, 161.0)
- moved P13 5.41 mm to (75.0, 161.0)
- moved P14 5.41 mm to (60.0, 161.0)
- moved P9 5.41 mm to (140.0, 161.0)
Routing:
- net +3V3: track 387.1 -> 399.6 mm, vias 2 -> 4
- net /RightW: track 54.6 -> 46.3 mm
- net GND: track 558.3 -> 551.1 mm
- net /RightV: track 41.3 -> 34.2 mm
- net /RightU: track 27.9 -> 22.2 mm
- net /LeftW: track 30.9 -> 34.2 mm
- net /LeftV: track 44.5 -> 46.2 mm
- net /LeftU: track 57.5 -> 58.1 mm
- added copper zone on B.Cu, net +3V3
