File: Circuit/MainControl/rhand_controller.kicad_pcb (KiCad board)
At the start: 2 copper layers, 100 x 100 mm, 43 parts, among them P1 BLUETOOTH, P10 LV_ADC, P11 LW_ADC, P12 RU_ADC, P13 RV_ADC, P14 RW_ADC, P2 CONN_01X06, P3 Wall, P4 CW, P5 Enable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

Commit message: メイン基板の変更とジョイスティック固定用基板の作成
Routing:
- net /SWO: track 4.29 -> 9.24 mm
- net /SWDIO: track 8.33 -> 13.2 mm
- net /SWCLK: track 5.68 -> 10.5 mm
- net /NRST: track 8.59 -> 13.3 mm
- added copper zone on B.Cu, net GND
- added copper zone on B.Cu, net Net-(BT1-Pad1)
Changed lines of the file:
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@@
     (thickness 1.6)
     (drawings 9)
-    (tracks 354)
+    (tracks 362)
     (zones 0)
     (modules 43)
@@
   )
   (setup
-    (last_trace_width 0.5)
+    (last_trace_width 1.5)
     (user_trace_width 0.4)
     (user_trace_width 1)
@@
   (segment (start 93.6 136.75) (end 93.6 154.9) (width 0.5) (layer B.Cu) (net 17) (status 10))
   (segment (start 92.5 156) (end 90 156) (width 0.5) (layer B.Cu) (net 17))
+  (segment (start 82.34 74.05) (end 82.34 75.34) (width 0.5) (layer B.Cu) (net 18))
+  (segment (start 82.34 75.34) (end 82.34 78.84) (width 1.5) (layer B.Cu) (net 18))
   (segment (start 89.75 129.7) (end 88.95 129.7) (width 0.5) (layer B.Cu) (net 18))
   (segment (start 86.95 127.7) (end 86.95 125.65) (width 1.5) (layer B.Cu) (net 18))
   (segment (start 88.95 129.7) (end 86.95 127.7) (width 0.5) (layer B.Cu) (net 18))
+  (segment (start 87.42 74.05) (end 87.42 74.92) (width 0.5) (layer B.Cu) (net 19) (status 400000))
+  (segment (start 87.42 74.92) (end 87.42 78.92) (width 1.5) (layer B.Cu) (net 19))
   (segment (start 89.75 130.5) (end 88.1 130.5) (width 0.5) (layer B.Cu) (net 19))
   (segment (start 85.25 126.75) (end 85.25 125) (width 1.5) (layer B.Cu) (net 19))
   (segment (start 85.25 127.65) (end 85.25 126.75) (width 0.5) (layer B.Cu) (net 19))
   (segment (start 88.1 130.5) (end 85.25 127.65) (width 0.5) (layer B.Cu) (net 19))
+  (segment (start 89.96 74.05) (end 89.96 75.46) (width 0.5) (layer B.Cu) (net 20) (status 400000))
+  (segment (start 89.96 75.46) (end 89.96 78.759998) (width 1.5) (layer B.Cu) (net 20))
   (segment (start 100.85 132.1) (end 100.85 132.5) (width 0.5) (layer B.Cu) (net 20))
   (segment (start 100.85 132.5) (end 102.2 132.5) (width 1.5) (layer B.Cu) (net 20))
@@
   (segment (start 105.03 132.1) (end 105.05 132.12) (width 0.5) (layer B.Cu) (net 20))
   (segment (start 98.27 132.12) (end 98.25 132.1) (width 0.5) (layer B.Cu) (net 20) (status 30))
+  (segment (start 92.5 74.05) (end 92.5 76) (width 0.5) (layer B.Cu) (net 21))
+  (segment (start 92.5 76) (end 92.5 79) (width 1.5) (layer B.Cu) (net 21))
   (segment (start 92 128.25) (end 92 127.35) (width 0.5) (layer B.Cu) (net 21))
   (segment (start 91.05 126.4) (end 89.6 124.95) (width 1.5) (layer B.Cu) (net 21))
@@
       )
     )
+  )
+  (zone (net 2) (net_name GND) (layer B.Cu) (hatch edge 0.508)
+    (connect_pads yes (clearance 0.508))
+    (min_thickness 0.254)
+    (fill yes (arc_segments 16) (thermal_gap 0.508) (thermal_bridge_width 0.508))
+    (polygon
+      (pts
+        (xy 110 81) (xy 104 81.5) (xy 104 73.5) (xy 110 73.5)
+      )
+    )
+  )
+  (zone (net 1) (net_name "Net-(BT1-Pad1)") (layer B.Cu) (hatch edge 0.508)
+    (connect_pads yes (clearance 0.508))
+    (min_thickness 0.254)
+    (fill yes (arc_segments 16) (thermal_gap 0.508) (thermal_bridge_width 0.508))
+    (polygon
+      (pts
+        (xy 126 75) (xy 124 75) (xy 124 74.5) (xy 121.5 74.5) (xy 121.5 77.5)
+        (xy 112 77.5) (xy 112 72) (xy 126 72)
+      )
+    )
