File: Circuit/MainControl/V1/rhand_controller.sch (KiCad schematic (older format))
At the start: 18 parts, among them P1 BLUETOOTH, SW1 EmSW, SW2 SWITCH_INV, U1 IM315TRX, U2 STM32F042

Commit message: フォルダ構造の変更
Connections:
- net Em_SW: now reaches R4.2, SW1.2, U2.25 (PA15/SPI1_NSS/I2S1_WS/USART2_RX/TIM2_CH1_ETR/EVENTOUT/USB_NOE)
Other:
- moved on the sheet: R4, SW1
Changed lines of the file:
@@
 LIBS:contrib
 LIBS:valves
-LIBS:YASU
 LIBS:device
 LIBS:rhand_controller-cache
@@
 L SW_PUSH SW1
 U 1 1 59392826
-P 2600 7200
-F 0 "SW1" H 2750 7310 50  0000 C CNN
-F 1 "EmSW" H 2600 7120 50  0000 C CNN
-F 2 "YASU:XA_2Pin" H 2600 7200 50  0001 C CNN
-F 3 "" H 2600 7200 50  0000 C CNN
-	1    2600 7200
+P 2450 7150
+F 0 "SW1" H 2600 7260 50  0000 C CNN
+F 1 "EmSW" H 2450 7070 50  0000 C CNN
+F 2 "YASU:XA_2Pin" H 2450 7150 50  0001 C CNN
+F 3 "" H 2450 7150 50  0000 C CNN
+	1    2450 7150
 	0    -1   -1   0
 $EndComp
@@
 L R R4
 U 1 1 5939354D
-P 2600 6600
-F 0 "R4" V 2680 6600 50  0000 C CNN
-F 1 "10k" V 2600 6600 50  0000 C CNN
-F 2 "Resistors_ThroughHole:R_Axial_DIN0207_L6.3mm_D2.5mm_P7.62mm_Horizontal" V 2530 6600 50  0001 C CNN
-F 3 "" H 2600 6600 50  0000 C CNN
-	1    2600 6600
-	1    0    0    -1
-$EndComp
-Wire Wire Line
-	2600 6750 2600 6900
-Connection ~ 2600 6850
-Wire Wire Line
-	2600 6450 2600 6350
-Wire Wire Line
-	2600 7500 2600 7600
+P 2450 6550
+F 0 "R4" V 2530 6550 50  0000 C CNN
+F 1 "10k" V 2450 6550 50  0000 C CNN
+F 2 "Resistors_ThroughHole:R_Axial_DIN0207_L6.3mm_D2.5mm_P7.62mm_Horizontal" V 2380 6550 50  0001 C CNN
+F 3 "" H 2450 6550 50  0000 C CNN
+	1    2450 6550
+	1    0    0    -1
+$EndComp
+Wire Wire Line
+	2450 6700 2450 6850
+Connection ~ 2450 6800
+Wire Wire Line
+	2450 6400 2450 6300
+Wire Wire Line
+	2450 7450 2450 7550
 $Comp
 L +3.3V #PWR018
 U 1 1 59394953
-P 2600 6350
-F 0 "#PWR018" H 2600 6200 50  0001 C CNN
-F 1 "+3.3V" H 2600 6490 50  0000 C CNN
-F 2 "" H 2600 6350 50  0000 C CNN
-F 3 "" H 2600 6350 50  0000 C CNN
-	1    2600 6350
+P 2450 6300
+F 0 "#PWR018" H 2450 6150 50  0001 C CNN
+F 1 "+3.3V" H 2450 6440 50  0000 C CNN
+F 2 "" H 2450 6300 50  0000 C CNN
+F 3 "" H 2450 6300 50  0000 C CNN
+	1    2450 6300
 	1    0    0    -1
 $EndComp
@@
 L GND #PWR019
 U 1 1 593949C5
-P 2600 7600
-F 0 "#PWR019" H 2600 7350 50  0001 C CNN
-F 1 "GND" H 2600 7450 50  0000 C CNN
-F 2 "" H 2600 7600 50  0000 C CNN
-F 3 "" H 2600 7600 50  0000 C CNN
-	1    2600 7600
+P 2450 7550
+F 0 "#PWR019" H 2450 7300 50  0001 C CNN
+F 1 "GND" H 2450 7400 50  0000 C CNN
+F 2 "" H 2450 7550 50  0000 C CNN
+F 3 "" H 2450 7550 50  0000 C CNN
+	1    2450 7550
 	1    0    0    -1
 $EndComp
@@
 $EndSheet
 Wire Wire Line
-	2600 6850 3100 6850
-Wire Wire Line
-	3100 6850 3100 6200
-Wire Wire Line
-	3100 6200 3250 6200
+	2450 6800 3150 6800
 $Sheet
 S 6250 2450 950  400
@@
 Wire Wire Line
 	9300 1500 9300 1400
+Text Label 2950 6800 2    60   ~ 0
+Em_SW
+Wire Wire Line
+	3150 6800 3150 6200
+Wire Wire Line
+	3150 6200 3250 6200
 $EndSCHEMATC
