File: Circuit/MainControl/V2/Left_Hand.sch (KiCad schematic (older format))
At the start: 2 parts, among them J2 L_Hand

Commit message: 回路設計完了
Connections:
- net Joy_X: now also J2.4 (P4); no longer J2.3 (P3)
- net Joy_Y: now also J2.3 (P3); no longer J2.4 (P4)
Changed lines of the file:
@@
 Wire Wire Line
 	4950 2600 4950 2550
-Text HLabel 5150 2950 2    60   Output ~ 0
+Text HLabel 5150 3050 2    60   Output ~ 0
 Joy_X
 Wire Wire Line
@@
 Wire Wire Line
 	4650 3150 5150 3150
-Text HLabel 5150 3050 2    60   Output ~ 0
+Text HLabel 5150 2950 2    60   Output ~ 0
 Joy_Y
 Text HLabel 5150 3150 2    60   Output ~ 0
